Commit message: longer time horizon

File: upright_assets/thing/xacro/obstacles/spheres.urdf.xacro (robot description, xacro)
@@ -4,5 +4,5 @@
     <link name="sphere_1">
         <collision>
-        <origin rpy="0 0 0" xyz="0.5 0 0.75"/>
+        <origin rpy="0 0 0" xyz="0.5 0 0.5"/>
         <geometry>
             <sphere radius="$(arg radius)"/>
@@ -10,5 +10,5 @@
         </collision>
         <visual>
-        <origin rpy="0 0 0" xyz="0.5 0 0.75"/>
+        <origin rpy="0 0 0" xyz="0.5 0 0.5"/>
         <geometry>
             <sphere radius="$(arg radius)"/>
@@ -17,5 +17,5 @@
         </visual>
     </link>
-    <link name="sphere_2">
+    <!-- <link name="sphere_2">
         <collision>
         <origin rpy="0 0 0" xyz="0.75 0.25 0.75"/>
@@ -46,5 +46,5 @@
         <material name="red"/>
         </visual>
-    </link>
+    </link> -->
     <link name="world"/>
     <joint name="fixed_joint_1" type="fixed">
@@ -53,5 +53,5 @@
         <origin rpy="0 0 0" xyz="0 0 0"/>
     </joint>
-    <joint name="fixed_joint_2" type="fixed">
+    <!-- <joint name="fixed_joint_2" type="fixed">
         <parent link="world"/>
         <child link="sphere_2"/>
@@ -62,4 +62,4 @@
         <child link="sphere_3"/>
         <origin rpy="0 0 0" xyz="0 0 0"/>
-    </joint>
+    </joint> -->
 </robot>
