Commit message: created panda subdir

File: upright_cmd/config/panda/assets/obstacles.urdf.xacro (robot description, xacro)
@@ -1,6 +1,6 @@
 <?xml version="1.0" ?>
-<robot name="spheres" xmlns:xacro="http://ros.org/wiki/xacro">
+<robot name="obstacles" xmlns:xacro="http://ros.org/wiki/xacro">
     <xacro:arg name="radius" default="0.1"/>
-    <link name="sphere_1">
+    <link name="static_1">
         <collision>
         <origin rpy="0 0 0" xyz="0.5 0 0.5"/>
@@ -17,5 +17,5 @@
         </visual>
     </link>
-    <!-- <link name="sphere_2">
+    <link name="static_2">
         <collision>
         <origin rpy="0 0 0" xyz="0.75 0.25 0.75"/>
@@ -32,5 +32,5 @@
         </visual>
     </link>
-    <link name="sphere_3">
+    <link name="static_3">
         <collision>
         <origin rpy="0 0 0" xyz="0.25 -0.25 0.25"/>
@@ -46,20 +46,20 @@
         <material name="red"/>
         </visual>
-    </link> -->
+    </link>
     <link name="world"/>
     <joint name="fixed_joint_1" type="fixed">
         <parent link="world"/>
-        <child link="sphere_1"/>
+        <child link="static_1"/>
         <origin rpy="0 0 0" xyz="0 0 0"/>
     </joint>
-    <!-- <joint name="fixed_joint_2" type="fixed">
+    <joint name="fixed_joint_2" type="fixed">
         <parent link="world"/>
-        <child link="sphere_2"/>
+        <child link="static_2"/>
         <origin rpy="0 0 0" xyz="0 0 0"/>
     </joint>
     <joint name="fixed_joint_3" type="fixed">
         <parent link="world"/>
-        <child link="sphere_3"/>
+        <child link="static_3"/>
         <origin rpy="0 0 0" xyz="0 0 0"/>
-    </joint> -->
+    </joint>
 </robot>
